File: KiCad/Servo_Driver.kicad_pcb (KiCad board)
At the start: 2 copper layers, 98.4 x 57.2 mm, 33 parts, among them J1 2Cell, J2 Servo_1, J3 Servo_2, J4 SIGNAL_INPUT, SW1 PWM1_SW, SW2 PWM2_SW, SW3 RST_SW, SW4 CENTER_SW, SW5 EN1_SW, SW6 EN2_SW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

Commit message: 基板を更新。部品配置の変更とフットプリントの配置
Parts:
- removed C5, C6, C7: 0.1u, Capacitor_THT:C_Disc_D4.3mm_W1.9mm_P5.00mm
- added G***: LOGO, Logos:Servodriver_TwinServo, F.Cu at (140.2, 117.1)
- added G***: LOGO, Logos:Musojin, F.Cu at (162.6, 99.1)
- added G***: LOGO, Logos:Musojin, B.Cu at (163.6, 99.1)
- added REF**: ESD-Logo_6.6x6mm_SilkScreen, Symbol:ESD-Logo_6.6x6mm_SilkScreen, F.Cu at (139.2, 73.9)
- G***: footprint Logos:Servodriver_suzuka_nega -> Logos:Servodriver_suzuka; moved to B.Cu
- moved C3 12.3 mm to (137.9, 94.5)
- moved C2 8.88 mm to (132.3, 80.0)
- moved G*** 7.06 mm to (136.1, 114.6), turned to 180 degrees
- moved J4 4.44 mm to (104.8, 111.1)
- moved C4 2.57 mm to (139.6, 100.8)
- moved D1 1.40 mm to (127.5, 79.5)
Routing:
- net /PWM2_IN: track 22.0 -> 26.5 mm
- net /PWM1_IN: track 22.5 -> 26.9 mm
- net /EN1: track 17.5 -> 14.4 mm
- net /CENTER: track 24.1 -> 21.0 mm
- net /EN2: track 32.4 -> 30.2 mm
- net GND: vias 0 -> 4
Other:
- board text added: "GND"
- board text added: "Musojin_Servo-Driver v0.1"
- board text added: "PWM1_IN"
- board text added: "PWM2_IN"
- board text added: "Produced by Seyanaga"

Commit message: 基板にシルクスクリーンを追加、その他位置を微調整
Other:
- board text added: "Produced by S.Miyazato"
- board text removed: "Produced by Seyanaga"
